File: pcb/Solaranimal210330_1217/Solaranimal210330_1217.kicad_pcb (KiCad board)
At the start: 2 copper layers, 78 x 32 mm, 26 parts, among them J1 Conn_01x01, J2 Conn_01x01, J3 Conn_01x01, J4 Conn_01x01, M3 MountingHole_3.2mm_M3_Pad_Top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, Q1 2N7000, Q2 BS170, SW1 SW_SPDT, SW2 SW_Push_standard_6x6_four_pins, U1 YX8051_JF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

Commit message: change pcb to new version
Parts:
- R1: value 1,5M -> 1M
- R2: value 470k -> 330k
- R3: value 470k -> 510k
- moved M3 4.00 mm to (98.0, 54.0)
Routing:
- net Net-(R7-Pad2): track 34.7 -> 41.5 mm
- net Net-(J4-Pad1): track 50.6 -> 48.5 mm
Other:
- board text added: "2021"
- board text added: "RESET"
- board text added: "V1.011"
- board text added: "open source hardware: github.com/kazoosh"
- board text removed: "R"
