File: pcb/Solaranimal210330_1217/Solaranimal210330_1217.kicad_pcb (KiCad board)
At the start: 2 copper layers, 78 x 32 mm, 26 parts, among them J1 Conn_01x01, J2 Conn_01x01, J3 Conn_01x01, J4 Conn_01x01, M3 MountingHole_3.2mm_M3_Pad_Top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, Q1 2N7000, Q2 BS170, SW1 SW_SPDT, SW2 SW_Push_standard_6x6_four_pins, U1 YX8051_JF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

Commit message: minor changes
Other:
- board text added: "V1.012"
- board text removed: "V1.011"

Commit message: change Q2
Parts:
- Q2: value BS170 -> ZVN4206AVSTZ
