File: pcb/Solaranimal210330_1217/Solaranimal210330_1217.sch (KiCad schematic (older format))
At the start: 26 parts, among them J1 Conn_01x01, J2 Conn_01x01, J3 Conn_01x01, J4 Conn_01x01, Q1 2N7000, Q2 BS170, SW1 SW_SPDT, SW2 SW_Push_standard_6x6_four_pins, U1 YX8051_JF, U2 ATtiny85V-10PU

Commit message: change pcb to new version
Parts:
- R1: value 1,5M -> 1M
- R2: value 470k -> 330k
- R3: value 470k -> 510k
Changed lines of the file:
@@
 encoding utf-8
 Sheet 1 1
-Title "Solaranimal210329_1841"
-Date "2021-03-29"
-Rev "1.01"
+Title "Solaranimal210330_1217"
+Date "2021-03-30"
+Rev "1.011"
 Comp "KAZOOSH!"
-Comment1 "(version with Reset-Button and changed LED connection)"
+Comment1 "V1.011(new R values, RESET-SW and changed LED connection)"
 Comment2 "2.5.2021 to 9.5.2021"
 Comment3 "wochedesgutenlebens.de"
-Comment4 ""
+Comment4 "open hardware: github.com/kazoosh"
 $EndDescr
 $Comp
@@
 P 2650 2900
 F 0 "R3" H 2720 2946 50  0000 L CNN
-F 1 "470k" H 2720 2855 50  0000 L CNN
+F 1 "510k" H 2720 2855 50  0000 L CNN
 F 2 "Resistor_THT:R_Axial_DIN0207_L6.3mm_D2.5mm_P10.16mm_Horizontal" V 2580 2900 50  0001 C CNN
 F 3 "~" H 2650 2900 50  0001 C CNN
@@
 P 2200 2900
 F 0 "R1" H 2270 2946 50  0000 L CNN
-F 1 "1,5M" H 2270 2855 50  0000 L CNN
+F 1 "1M" H 2270 2855 50  0000 L CNN
 F 2 "Resistor_THT:R_Axial_DIN0207_L6.3mm_D2.5mm_P10.16mm_Horizontal" H 2270 2809 50  0001 L CNN
 F 3 "~" H 2200 2900 50  0001 C CNN
@@
 P 2200 4400
 F 0 "R2" H 2270 4446 50  0000 L CNN
-F 1 "470k" H 2270 4355 50  0000 L CNN
+F 1 "330k" H 2270 4355 50  0000 L CNN
 F 2 "Resistor_THT:R_Axial_DIN0207_L6.3mm_D2.5mm_P10.16mm_Horizontal" V 2130 4400 50  0001 C CNN
 F 3 "~" H 2200 4400 50  0001 C CNN
