File: pcb/Solaranimal210330_1217/Solaranimal210330_1217.sch (KiCad schematic (older format))
At the start: 26 parts, among them J1 Conn_01x01, J2 Conn_01x01, J3 Conn_01x01, J4 Conn_01x01, Q1 2N7000, Q2 BS170, SW1 SW_SPDT, SW2 SW_Push_standard_6x6_four_pins, U1 YX8051_JF, U2 ATtiny85V-10PU

Commit message: change Q2
Parts:
- removed Q2: BS170, Package_TO_SOT_THT:TO-92_Inline_Wide, symbol Transistor_FET:BS170
- added Q2: ZVN4206AVSTZ, Package_TO_SOT_THT:TO-92_Inline_Wide, symbol Joe_Library:ZVN4206AVSTZ
Connections:
- net GND: now also Q2.3 (S)
- net at J1.1 (Pin_1), R4.2, SC1.1 (+)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: now also Q2.1 (D)
- net at Q1.3 (D), R3.2: now also Q2.2 (G)
Changed lines of the file:
@@
 P 2550 4150
 F 0 "Q1" H 2700 4350 50  0000 L CNN
-F 1 "2N7000" H 2700 3950 50  0000 L CNN
+F 1 "2N7000" H 2550 3800 50  0000 L CNN
 F 2 "Package_TO_SOT_THT:TO-92_Inline_Wide" H 2750 4075 50  0001 L CIN
 F 3 "https://www.onsemi.com/pub/Collateral/NDS7002A-D.PDF" H 2550 4150 50  0001 L CNN
 	1    2550 4150
-	1    0    0    -1
-$EndComp
-$Comp
-L Transistor_FET:BS170 Q2
-U 1 1 6064E0A2
-P 3100 4150
-F 0 "Q2" H 3250 4350 50  0000 L CNN
-F 1 "BS170" H 3250 3950 50  0000 L CNN
-F 2 "Package_TO_SOT_THT:TO-92_Inline_Wide" H 3300 4075 50  0001 L CIN
-F 3 "https://www.onsemi.com/pub/Collateral/BS170-D.PDF" H 3100 4150 50  0001 L CNN
-	1    3100 4150
 	1    0    0    -1
 $EndComp
@@
 Wire Wire Line
 	7850 4050 9200 4050
+$Comp
+L Joe_Library:ZVN4206AVSTZ Q2
+U 1 1 606703B3
+P 3100 4150
+F 0 "Q2" H 3300 4350 50  0000 L CNN
+F 1 "ZVN4206AVSTZ" H 3050 3800 50  0000 L CNN
+F 2 "Package_TO_SOT_THT:TO-92_Inline_Wide" H 3300 4075 50  0001 L CIN
+F 3 "https://docs.rs-online.com/0ef4/0900766b81321be1.pdf" H 3100 4150 50  0001 L CNN
+	1    3100 4150
+	1    0    0    -1
+$EndComp
 $EndSCHEMATC
