File: circuit/Solaranimal210527_2049/Solaranimal210527_2049.sch (KiCad schematic (older format))
At the start: 28 parts, among them J1 Conn_01x01, J2 Conn_01x01, J3 Conn_01x01, J4 Conn_01x01, Q1 2N7000, Q2 BS170, SW1 SW_SPDT, SW2 SW_Push_standard_6x6_four_pins, U1 QX5252F, U2 ATtiny85V-10PU

Commit message: Update Solaranimal210527_2049.sch
Parts:
- added R8: 33k, Resistor_THT:R_Axial_DIN0207_L6.3mm_D2.5mm_P10.16mm_Horizontal, symbol Device:R
Connections:
- net GND: now also R8.2
- net at J1.1 (Pin_1), Q2.1 (D), R4.2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: now also R8.1
Other:
- note added: "10.) Zum Start Batterieschalter in Richtung PIEZO schieben und RESET drücken."
- note added: "9.) R8 wird durch J1 und J2 gesteckt und gelötet."
- note removed: "9.) Zum Start Batterieschalter in Richtung PIEZO schieben und RESET drücken."
- moved on the sheet: C3, Q1, Q2, R1, R2, R3, R4
